File: 3109-comparisons.sch (EAGLE design)
At the start: 152 parts, among them IC1 LM4558N, IC2 LM4558N, IC3 LM4558N, Q1 2SA1015, Q2 2SA1015-GR, Q3 2SA1015-GR, Q4 2SA1015, T3 2SC945, T4 2SC945

Commit message: Finished JP6 filter
Parts:
- added C27, C28, C29, C30: 330p, resistor:C-EU025-024X044
- added C31, C33: 5p, resistor:C-EU025-024X044
- added C32, C34: 33p, resistor:C-EU025-024X044
- added C35: 4n7, resistor:C-EU025-024X044
- added D1, D2: 1S24735, joakim:1S24735
- added IC4: M5218JL, joakim:M5218JL
- added IC5, IC6: MC14551JN, joakim:MC14551JN
- added R110, R112: 56k, resistor:R-US_0204/7
- added R111, R113, R115, R121, R122, R131, R144: 68k, resistor:R-US_0204/7
- added R114, R116, R127, R136: 10k, resistor:R-US_0204/7
- added R117, R118, R119, R120, R123, R132: 560R, resistor:R-US_0204/7
- added R124, R125, R130, R133, R134: 100k, resistor:R-US_0204/7
- added R126, R129, R135: 33k, resistor:R-US_0204/7
- added R128, R137: 47k, resistor:R-US_0204/7
- added R138: 100k, resistor:R-TRIMMT93XA
- added R139, R141: 1k2G, resistor:R-US_0204/7
- added R140: 130k, resistor:R-US_0204/7
- added R142: 180k, resistor:R-US_0204/7
- added R143, R146: 1M, resistor:R-US_0204/7
- added R145: 220k, resistor:R-US_0204/7
- added R147: 100kB, resistor:R-TRIMMT93XA
- added U$11: IR3109-OTA, joakim:IR3109-OTA
- added U$9: IR3109, joakim:IR3109
- U$8: value BA662-J -> IR9022; device joakim:BA662-J -> joakim:IR9022
Connections:
- removed net N$79: U$8G$1.C_BUFF
- new net N$120: R128.1, R129.1
- new net N$121: C27.1, U$9G$4.CAP
- new net N$122: R111.1, R122.1, R129.2, U$9G$4.OUT
- new net N$123: C30.1, U$9G$3.CAP
- new net N$124: R118.2, R121.2, U$9G$4.IN
- new net N$125: R111.2, R117.2, U$9G$1.IN
- new net N$126: C33.2, R114.1, R134.2, U$9G$3.OUT
- new net N$127: R113.2, R119.2, U$9G$2.IN
- new net N$128: C29.1, U$9G$2.CAP
- new net N$129: R115.2, R120.2, U$9G$3.IN
- new net N$130: R115.1, R131.1, R137.1, U$9G$2.OUT
- new net N$131: IC4A.OUT, R112.1, R121.1, R124.2
- new net N$132: IC4B.OUT, R113.1, R116.1, R133.2
- new net N$134: R122.2, R123.2, U$11G$4.IN
- new net N$135: C31.1, IC4A.-IN, R124.1, R125.1, U$11G$4.CAP
- new net N$136: C31.2, R110.1, R125.2, U$9G$1.OUT
- new net N$137: IC5G$5.CTRL
- new net N$138: IC5G$1.0, R110.2
- new net N$139: IC5G$1.1, R112.2
- new net N$140: IC6G$1.0, R114.2
- new net N$141: IC6G$1.1, R116.2
- new net N$142: IC5G$1.COM, R130.2
- new net N$143: IC6G$5.CTRL
- new net N$144: U$11G$5.CTRL
- new net N$145: R131.2, R132.2, U$11G$3.IN
- new net N$146: R138.S, R143.2
- new net N$147: C33.1, IC4B.-IN, R130.1, R133.1, R134.1
- new net N$148: D1.A, D2.C, R136.2, R137.2
- new net N$149: C34.2, D1.C, D2.A, IC4B.+IN, R135.2
- new net N$150: R140.1
- new net N$151: C32.2, IC4A.+IN, R126.2, R127.2, R128.2
- new net N$152: C35.2, R139.1, U$9G$5.CTRL
- new net N$153: R139.2, R144.2, R145.1, R146.2, U$8G$2.-IN, U$8G$2.OUT
- new net N$154: R140.2, R141.2, R142.2, R143.1
- new net N$155: C35.1, R144.1
- new net N$156: R146.1, R147.S
- new net N$57: C28.1, U$9G$1.CAP
- net +15V: now also R138.A, R147.A; no longer U$1G$6.+V, U$3G$6.+V, U$5G$6.+V, U$7G$6.+V, U$8G$1.IN_BUFF, U$8G$3.V+
- net -15V: now also R138.E, R142.1, R145.2, R147.E; no longer U$1G$6.-V, U$3G$6.-V, U$5G$6.-V, U$7G$6.-V, U$8G$3.V-
- net GND: now also C27.2, C28.2, C29.2, C30.2, C32.1, C34.1, R117.1, R118.1, R119.1, R120.1, R123.1, R126.1, R127.1, R132.1, R135.1, R136.1, R141.1, U$8G$2.+IN; no longer U$1G$6.GND, U$3G$6.GND, U$5G$6.GND, U$7G$6.GND
- net N$64: now also U$4G$2.C_OTA
Other:
- note added: "7k7 combined"
- note added: "JP6"
- note added: "Latch 12"
- note added: "Latch 15"
- note added: "Posistor"

Commit message: New version
Parts:
- added C36, C37, C38, C39: 330p, resistor:C-EU025-024X044
- added C40, C42: 5p, resistor:C-EU025-024X044
- added C41, C43: 33p, resistor:C-EU025-024X044
- added D3, D4: 1S24735, joakim:1S24735
- added IC7: M5218JL, joakim:M5218JL
- added IC8: M5218, joakim:M5218JL
- added R148, R149, R150, R155, R160, R169, R178: 68k, resistor:R-US_0204/7
- added R151, R152, R153, R154, R161, R170: 560R, resistor:R-US_0204/7
- added R156: 56k, resistor:R-US_0204/7
- added R157: 130k, resistor:R-US_0204/7
- added R158, R181: 1k2G, resistor:R-US_0204/7
- added R159: 180k, resistor:R-US_0204/7
- added R162, R163, R168, R171, R172: 100k, resistor:R-US_0204/7
- added R164, R167, R173: 33k, resistor:R-US_0204/7
- added R165, R174: 10k, resistor:R-US_0204/7
- added R166, R175: 47k, resistor:R-US_0204/7
- added R176, R179: 1M, resistor:R-US_0204/7
- added R177: 100k, resistor:R-TRIMMT93XA
- added R180: 100kB, resistor:R-TRIMMT93XA
- added R182: 107k, resistor:R-US_0204/7
- added U$10, U$13: IR3109, joakim:IR3109
- added U$12, U$14: IR3109-OTA, joakim:IR3109-OTA
Connections:
- new net -8V: R182.2
- new net N$133: R148.2, R151.2, U$10G$1.IN
- new net N$157: R149.2, R153.2, U$10G$2.IN
- new net N$158: R150.2, R154.2, U$10G$3.IN
- new net N$159: R156.2, R168.2
- new net N$160: IC7B.OUT, R149.1, R171.2
- new net N$161: R160.2, R161.2, R167.2, U$12G$4.IN
- new net N$162: C37.1, U$10G$1.CAP
- new net N$163: C36.1, U$10G$4.CAP
- new net N$164: R148.1, R160.1, U$10G$4.OUT
- new net N$165: C39.1, U$10G$3.CAP
- new net N$166: C42.2, R172.2, U$10G$3.OUT
- new net N$167: C38.1, U$10G$2.CAP
- new net N$168: R150.1, R169.1, R175.1, U$10G$2.OUT
- new net N$169: C40.1, IC7A.-IN, R162.1, R163.1, U$12G$4.CAP
- new net N$170: C40.2, R156.1, R163.2, U$10G$1.OUT
- new net N$171: R166.1, R167.1
- new net N$172: IC7A.OUT, R155.1, R162.2
- new net N$173: U$14G$5.CTRL
- new net N$174: R157.2, R158.2, R159.2, R176.1
- new net N$175: R176.2, R177.S
- new net N$176: R157.1
- new net N$177: R169.2, R170.2, U$12G$3.IN
- new net N$178: C42.1, IC7B.-IN, R168.1, R171.1, R172.1, U$12G$3.CAP
- new net N$179: D3.A, D4.C, R174.2, R175.2
- new net N$180: C43.2, D3.C, D4.A, IC7B.+IN, R173.2
- new net N$181: C41.2, IC7A.+IN, R164.2, R165.2, R166.2
- new net N$182: R179.1, R180.S
- new net N$183: IC8B.-IN, R179.2, R181.2, R182.1
- new net N$185: R178.1, R181.1, U$13G$5.CTRL
- new net N$186: C35.1, R144.2, U$8G$2.OUT
- new net N$79: R152.2, R155.2, U$10G$4.IN
- net +15V: now also R177.A, R180.A
- net -15V: now also R159.1, R177.E, R180.E
- net GND: now also C36.2, C37.2, C38.2, C39.2, C41.1, C43.1, IC8B.+IN, R151.1, R152.1, R153.1, R154.1, R158.1, R161.1, R164.1, R165.1, R170.1, R173.1, R174.1
- net N$122: no longer R129.2
- net N$134: now also R129.2
- net N$152: now also R144.1; no longer C35.2
- net N$153: now also C35.2; no longer R144.2, U$8G$2.OUT
- net N$155: now also IC8B.OUT, R178.2; no longer C35.1, R144.1
Other:
- note added: "MKS-80"

Commit message: Added SH-101
Parts:
- added C44, C45, C46, C47: 240p, resistor:C-EU025-024X044
- added C48: 10u/16 BP, resistor:C-EU025-024X044
- added C50: 2u2 50V, resistor:CPOL-EUE2-5
- added C51, C52: 10u/16, resistor:CPOL-EUE2-5
- added D7, D8: 1S24735, joakim:1S24735
- added IC9: IR9022, linear:LM4558N
- added R183, R184, R185, R186, R187, R188, R189: 68k, resistor:R-US_0204/7
- added R190, R191, R192, R193: 560R, resistor:R-US_0204/7
- added R194, R195: 150k, resistor:R-US_0204/7
- added R196: 100K lin, resistor:R-TRIMMT93XA
- added R198, R217: 15k, resistor:R-US_0204/7
- added R199: 1k, resistor:R-US_0204/7
- added R200: ?, resistor:R-US_0204/7
- added R201: 820, resistor:R-US_0204/7
- added R202: SDT-1000, resistor:R-US_0204/7
- added R203: 1k8, resistor:R-US_0204/7
- added R204: 4k7, resistor:R-US_0204/7
- added R205: 33k, resistor:R-US_0204/7
- added R206, R216: 5k6, resistor:R-US_0204/7
- added R207: 680k, resistor:R-US_0204/7
- added R208: 2k2, resistor:R-US_0204/7
- added R209: 2M2, resistor:R-US_0204/7
- added R210: 47k, resistor:R-TRIMMT93XA
- added R211: 22k, resistor:R-US_0204/7
- added R215: 10k, resistor:R-US_0204/7
- added T1, T2, T5, T6: 2SC945, transistor:2SC945
- added U$15: IR3109, joakim:IR3109
- added U$16: BA662-J, joakim:BA662-J
Connections:
- new net IR3109_PIN_1: C44.2, C45.2, C46.2, C47.2, C50.+, D7.C, D8.A, R190.1, R191.1, R192.1, R193.1, R201.1
- new net N$184: C44.1, U$15G$1.CAP
- new net N$187: C45.1, U$15G$2.CAP
- new net N$188: C46.1, U$15G$3.CAP
- new net N$189: C47.1, U$15G$4.CAP
- new net N$190: R183.2, R184.1, U$15G$1.OUT
- new net N$192: R184.2, R185.1, R190.2, U$15G$2.IN
- new net N$193: R185.2, R186.1, U$15G$2.OUT
- new net N$194: R186.2, R187.1, R192.2, U$15G$3.IN
- new net N$195: R187.2, R188.1, U$15G$3.OUT
- new net N$196: R188.2, R189.1, R193.2, U$15G$4.IN
- new net N$197: R196.S, T5.B
- new net N$198: R189.2, R195.1, R196.A, U$15G$4.OUT
- new net N$199: R194.1, R215.2, T5.E
- new net N$200: C48.2, R183.1, R191.2, R217.2, U$15G$1.IN
- new net N$201: U$16G$1.C_BUFF
- new net N$202: C51.+, R198.2, R199.2, T6.C
- new net N$203: R194.2, R195.2
- new net N$204: C52.+, R200.1, T6.E
- new net N$205: C52.-, R216.1
- new net N$206: C48.1
- new net N$207: IC9B.-IN, R205.2
- new net N$208: R201.2, R202.1, R206.1, R207.1, U$15G$5.CTRL
- new net N$209: R202.2, R203.1
- new net N$210: R203.2, R204.1, R206.2
- new net N$212: IC9B.OUT, R204.2, R205.1
- new net N$214: R208.2, T2.C
- new net N$215: T1.E, T2.E
- new net N$216: R209.2, T1.B, T2.B
- new net N$217: R209.1, R210.S
- new net N$218: R210.E, R211.1
- new net N$220: R198.1, T5.C, T6.B
- new net N$222: D7.A, D8.C, R216.2, R217.1
- net +15V: now also R199.1, R207.2, U$16G$1.IN_BUFF, U$16G$3.V+
- net -15V: now also U$16G$3.V-
- net GND: now also C50.-, C51.-, IC9B.+IN, R200.2, R208.1, R211.2, R215.1
Other:
- note added: "Connected to "center ground" as synth is unipolar"
- note added: "SH-101"
- note added: "TODO: MC202, MKS30"

Commit message: Added MC-202
Parts:
- removed R210: 47k, resistor:R-TRIMMT93XA
- removed R211: 22k, resistor:R-US_0204/7
- removed T1, T2: 2SC945, transistor:2SC945
- removed U$16: BA662-J, joakim:BA662-J
- added C49, C53, C54, C55: 250p, resistor:C-EU025-024X044
- added C56: 10u/16 BP, resistor:C-EU025-024X044
- added C57: 47u/16V, resistor:CPOL-EUE2-5
- added C58, C59, C60: 10u/16, resistor:CPOL-EUE2-5
- added D5, D6: 1S24735, joakim:1S24735
- added IC10: TL022CP, linear:LM4558N
- added R197, R212, R213, R214, R218, R219, R220: 68k, resistor:R-US_0204/7
- added R221, R222, R223, R224: 560R, resistor:R-US_0204/7
- added R225, R226, R237: 150k, resistor:R-US_0204/7
- added R227: SDT-1000, resistor:R-US_0204/7
- added R228: 1k8, resistor:R-US_0204/7
- added R229, R238: 10k, resistor:R-US_0204/7
- added R230: 33k, resistor:R-US_0204/7
- added R231: 5k6, resistor:R-US_0204/7
- added R232: 680k, resistor:R-US_0204/7
- added R239: 100K lin, resistor:R-TRIMMT93XA
- added R241: 1k, resistor:R-US_0204/7
- added R243: 2k2, resistor:R-US_0204/7
- added R244: 15k, resistor:R-US_0204/7
- added R245: 3k3, resistor:R-US_0204/7
- added R246: 22k, resistor:R-US_0204/7
- added T10: 2SC945, transistor:2SC945
- added U$17: IR3109, joakim:IR3109
- R208: value 2k2 -> 15k
- R209: value 2M2 -> 10k
- T5, T6: value 2SC945 -> 2SC1815GR
Connections:
- removed net N$214: R208.2, T2.C
- removed net N$215: T1.E, T2.E
- removed net N$216: R209.2, T1.B, T2.B
- removed net N$217: R209.1, R210.S
- removed net N$218: R210.E, R211.1
- new net +12V: R241.1
- new net -5V: R238.2
- new net N$191: C49.1, U$17G$1.CAP
- new net N$211: C53.1, U$17G$2.CAP
- new net N$213: C54.1, U$17G$3.CAP
- new net N$219: C55.1, U$17G$4.CAP
- new net N$221: R197.2, R212.1, U$17G$1.OUT
- new net N$223: R212.2, R213.1, R221.2, U$17G$2.IN
- new net N$224: R213.2, R214.1, U$17G$2.OUT
- new net N$225: R214.2, R218.1, R223.2, U$17G$3.IN
- new net N$226: R218.2, R219.1, U$17G$3.OUT
- new net N$227: R219.2, R220.1, R224.2, U$17G$4.IN
- new net N$228: C56.2, R197.1, R222.2, R244.2, U$17G$1.IN
- new net N$230: C56.1
- new net N$231: IC10B.-IN, R230.2
- new net N$232: R226.2, R227.1, R231.1, R232.1, U$17G$5.CTRL
- new net N$233: R227.2, R228.1
- new net N$234: R228.2, R229.1, R231.2
- new net N$235: IC10B.OUT, R229.2, R230.1
- new net N$241: R220.2, R237.1, R239.A, U$17G$4.OUT
- new net N$242: R225.2, R237.2
- new net N$243: C60.+, R225.1, R239.S
- new net N$244: R209.2, R238.1, T10.E
- new net N$245: C60.-, R245.1
- new net N$246: C58.+, C59.+, R208.2, R241.2
- new net N$248: C59.-, R243.1
- new net N$249: D5.A, D6.C, R243.2, R244.1
- new net N$250: R245.2, R246.1, T10.B
- net +15V: now also R232.2; no longer U$16G$1.IN_BUFF, U$16G$3.V+
- net -15V: no longer U$16G$3.V-
- net GND: now also C57.-, C58.-, IC10B.+IN, R209.1, R246.2; no longer R208.1, R211.2
- net IR3109_PIN_1: now also C49.2, C53.2, C54.2, C55.2, C57.+, D5.C, D6.A, R221.1, R222.1, R223.1, R224.1, R226.1, R239.E
- net N$201: now also R208.1, T10.C; no longer U$16G$1.C_BUFF
Other:
- note added: "MC-202"
